Commit message: Trying to sort out joint state publisher

File: src/omnidrone_description/urdf/omnidrone.xacro (robot description, xacro)
@@ -109,4 +109,5 @@
   <child link="wheelFL_1"/>
   <axis xyz="-1.0 -0.0 -0.0"/>
+  <dynamics damping="0.5" friction="0.5" />
 </joint>
 <joint name="Revolute 2" type="continuous">
@@ -115,4 +116,5 @@
   <child link="wheelFR_1"/>
   <axis xyz="1.0 -0.0 -0.0"/>
+  <dynamics damping="0.5" friction="0.5" />
 </joint>
 <joint name="Revolute 3" type="continuous">
@@ -121,4 +123,5 @@
   <child link="wheelRR_4"/>
   <axis xyz="1.0 -0.0 -0.0"/>
+  <dynamics damping="0.5" friction="0.5" />
 </joint>
 <joint name="Revolute 4" type="continuous">
@@ -127,4 +130,5 @@
   <child link="wheelRL_1"/>
   <axis xyz="-1.0 -0.0 -0.0"/>
+  <dynamics damping="0.5" friction="0.5" />
 </joint>
 </robot>
